File: flex/flex.kicad_pcb (KiCad board)
At the start: 2 copper layers, 48.8 x 41.5 mm, 20 parts, among them J1 Conn_01x06_Female, J2 Conn_01x03_Female, SW19 SW_Push, SW5 SW_Push, SW9 SW_Push

Commit message: work
Parts:
- D10, D12, D2: footprint libs2:YS-SK6812MINI-E_REVERSE -> customs:SK6812_mini_e_corners
- D11, D13, D3: footprint libs2:YS-SK6812MINI-E_REVERSE_NO_EDGECUT -> customs:SK6812_mini_e_corners_noedgecuts
- moved D2 9.34 mm to (74.6, 93.7), turned to -170 degrees
- moved D3 9.34 mm to (74.6, 93.7), turned to -170 degrees
- moved D10 9.25 mm to (94.3, 69.9), turned to 180 degrees
- moved D11 9.25 mm to (94.3, 69.9), turned to 180 degrees
- moved D19 8.99 mm to (100.2, 65.5)
- moved D12 8.93 mm to (73.3, 72.0), turned to -170 degrees
- moved D13 8.93 mm to (73.3, 72.0), turned to -170 degrees
- turned SW19 to 180 degrees
- turned SW5 to -170 degrees
- turned SW9 to -170 degrees
Connections:
- D10 pad 1: Net-(D10-Pad1) -> Net-(D10-DOUT)
- D10 pad 3: Net-(D12-Pad1) -> (no net)
- D11 pad 1: Net-(D10-Pad1) -> Net-(D10-DOUT)
- D11 pad 3: Net-(D12-Pad1) -> Net-(D10-DIN)
- D12 pad 1: Net-(D12-Pad1) -> Net-(D10-DIN)
- D12 pad 3: Net-(D12-Pad3) -> (no net)
- D13 pad 1: Net-(D12-Pad1) -> Net-(D10-DIN)
- D13 pad 3: Net-(D12-Pad3) -> Net-(D12-DIN)
- D2 pad 1: unconnected-(D2-Pad1) -> (no net)
- D2 pad 3: Net-(D10-Pad1) -> (no net)
- D3 pad 1: unconnected-(D3-Pad1) -> (no net)
- D3 pad 3: Net-(D10-Pad1) -> Net-(D10-DOUT)
- R1 pad 1: Net-(D12-Pad3) -> Net-(D12-DIN)
- R2 pad 1: Net-(D12-Pad3) -> Net-(D12-DIN)
Routing:
- net Vcc: track 87.1 -> 0.00 mm, vias 4 -> 0
- net Gnd: track 77.7 -> 0.00 mm, vias 4 -> 0
- net Net-(D10-Pad1): track 69.9 -> 0.00 mm, vias 3 -> 0
- net row1: track 57.9 -> 0.00 mm, vias 2 -> 0
- net col6: track 56.4 -> 0.00 mm, vias 3 -> 0
- net Net-(D12-Pad1): track 28.0 -> 0.00 mm, vias 3 -> 0
- net Din: track 26.4 -> 0.00 mm, vias 1 -> 0
- net col4: track 20.2 -> 0.00 mm, vias 1 -> 0
- net Net-(D12-Pad3): track 19.5 -> 0.00 mm, vias 3 -> 0
- net Net-(D19-A): track 13.1 -> 0.00 mm, vias 1 -> 0
- net col2: track 12.7 -> 0.00 mm, vias 1 -> 0
- net Net-(D9-A): track 8.50 -> 0.00 mm, vias 1 -> 0
- net Net-(D5-A): track 6.63 -> 0.00 mm
Other:
- board text added: "GITHUB.COM/BASTARDKB BASTARDKB.COM"
- board text added: "Gnd"
- board text added: "Licensed under CC BY-NC-SA 4.0 Copyright Q. Lebastard 2025"
- board text added: "REV 3.0"
- board text added: "nano/mini"
- board text removed: "3 ROWS"
- board text removed: "BASTARDKB.COM"
- board text removed: "C2R5"
- board text removed: "C3R5"
- board text removed: "C5R5"
- board text removed: "CHARYBDIS THUMB CLUSTER"
- board text removed: "GITHUB.COM/BASTARDKB"
- board text removed: "Licensed under CC BY-NC-SA 4.0 Copyright Quentin Lebastard 2022"
- board text removed: "REV 2.01"

Commit message: routing
Routing:
- net Gnd: track 0.00 -> 109.5 mm, vias 0 -> 7
- net Vcc: track 0.00 -> 76.8 mm, vias 0 -> 4
- net row1: track 0.00 -> 51.0 mm, vias 0 -> 2
- net col6: track 0.00 -> 36.0 mm, vias 0 -> 2
- net Din: track 0.00 -> 27.0 mm, vias 0 -> 2
- net col4: track 0.00 -> 20.9 mm, vias 0 -> 1
- net Net-(D9-A): track 0.00 -> 19.9 mm, vias 0 -> 1
- net Net-(D12-DIN): track 0.00 -> 17.3 mm, vias 0 -> 2
- net Net-(D5-A): track 0.00 -> 14.6 mm, vias 0 -> 1
- net Net-(D19-A): track 0.00 -> 13.7 mm, vias 0 -> 1
- net col2: track 0.00 -> 13.6 mm, vias 0 -> 1
Other:
- board text added: "X"
- board text removed: "C3"
- board text removed: "C5"

Commit message: DRC
Parts:
- added Mousebite1: ~, customs:mousebite, F.Cu at (64.3, 78.2)
- added Mousebite2: ~, customs:mousebite, F.Cu at (101.5, 77.9)
- added Mousebite3: ~, customs:mousebite, F.Cu at (67.4, 99.7)
- added Mousebite4: ~, customs:mousebite, F.Cu at (87.2, 96.6)
Connections:
- D10 pad 3: (no net) -> Net-(D10-DIN)
- D12 pad 3: (no net) -> Net-(D12-DIN)
- D2 pad 1: (no net) -> unconnected-(D2-DOUT-Pad1)
- D2 pad 3: (no net) -> Net-(D10-DOUT)
- D3 pad 1: (no net) -> unconnected-(D3-DOUT-Pad1)
Routing:
- net Net-(D10-DIN): track 0.00 -> 51.1 mm, vias 0 -> 4
- net Net-(D10-DOUT): track 0.00 -> 45.0 mm, vias 0 -> 3
- net Net-(D12-DIN): track 17.3 -> 20.9 mm
- net col4: track 20.9 -> 22.9 mm
- net Vcc: track 76.8 -> 77.4 mm
- net Gnd: track 109.5 -> 110.1 mm
Other:
- outline, holes or cut-outs redrawn
